File: PCB_Chessboard/PCB_Quadrant/Connector.kicad_sch (KiCad schematic)
At the start: 48 parts, among them J10 Conn_01x02, J11 Conn_01x02, J12 Conn_01x02, J13 Conn_01x02, J14 Conn_01x02, J15 Conn_01x02, J16 Conn_01x02, J17 Conn_01x02, J18 Conn_01x02, J19 Conn_01x03, J2 Conn_01x02, J20 Conn_01x03, J3 Conn_01x02, J4 Conn_01x02, J5 Conn_01x02, J6 Conn_01x02, J7 Conn_01x02, J8 Conn_01x02, J9 Conn_01x02, Q1 BSS84

Commit message: PCB quadrant finalisé
Parts:
- removed H1, H2, H3, H4: MountingHole, MountingHole:MountingHole_4mm, symbol Mechanical:MountingHole
- removed J10, J11, J12, J13, J14, J15, J16, J17, J2, J3, J4, J5, J6, J7, J8, J9: Conn_01x02, Connector_PinHeader_2.54mm:PinHeader_1x02_P2.54mm_Vertical, symbol Connector_Generic:Conn_01x02
- C20, C21, C22, C23, C24, C25, C26, C27, C28, C29, C30, C31, C32, C4, C5, C6: value 47 pF -> 180 pF
- JP1, JP2, JP3, JP4, JQ1: footprint Connector_JST:JST_VH_B7PS-VH_1x07_P3.96mm_Horizontal -> Connector_JST:JST_XH_B7B-XH-A_1x07_P2.50mm_Vertical
Connections:
- net ANT1+: now also C20.1, C20.2, C21.1, C21.2, C22.1, C22.2, C23.1, C23.2, C24.1, C24.2, C4.1, C4.2, C5.1, C5.2, C6.1, C6.2
- net ANT10+: now also C25.1, C25.2, C26.1, C26.2, C27.1, C27.2, C28.1, C28.2, C29.1, C29.2, C30.1, C30.2, C31.1, C31.2, C32.1, C32.2
- net GND: no longer C20.2, C21.2, C22.2, C23.2, C24.2, C25.2, C26.2, C27.2, C28.2, C29.2, C30.2, C31.2, C32.2, C4.2, C5.2, C6.2
Other:
- moved on the sheet: C20, C21, C22, C23, C24, C25, C26, C27, C28, C29, C30, C31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
