File: PCB_Chessboard/PCB_Quadrant/PCB_Chessboard.kicad_pcb (KiCad board)
At the start: 4 copper layers, 200 x 200 mm, 79 parts, among them J10 Conn_01x02, J11 Conn_01x02, J12 Conn_01x02, J13 Conn_01x02, J14 Conn_01x02, J15 Conn_01x02, J16 Conn_01x02, J17 Conn_01x02, J18 Conn_01x02, J19 Conn_01x03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

Commit message: PCB quadrant finalisé
Parts:
- removed H1, H2, H3, H4: MountingHole, MountingHole:MountingHole_4mm
- removed J10, J11, J12, J13, J14, J15, J16, J17, J2, J3, J4, J5, J6, J7, J8, J9: Conn_01x02, Connector_PinHeader_2.54mm:PinHeader_1x02_P2.54mm_Vertical
- C20, C21, C22, C23, C24, C25, C26, C27, C28, C29, C30, C31, C32, C4, C5, C6: value 47 pF -> 180 pF
- JQ1: footprint Connector_JST:JST_VH_B7PS-VH_1x07_P3.96mm_Horizontal -> Connector_JST:JST_XH_B7B-XH-A_1x07_P2.50mm_Vertical
- moved C3 71.6 mm to (81.0, 16.0), turned to -90 degrees
- moved JQ1 63.6 mm to (99.5, 11.0), turned to -90 degrees
- moved Q1 59.3 mm to (85.0, 16.0)
- moved R1 58.6 mm to (82.4, 16.5)
- moved U3 57.4 mm to (100.0, 39.0)
- moved C2 56.5 mm to (108.6, 17.7)
- moved J18 56.5 mm to (112.6, 22.2)
- moved J19 56.2 mm to (112.5, 10.4)
- moved J20 56.0 mm to (91.0, 25.5)
- moved C9 51.6 mm to (94.5, 15.5), turned to 0 degrees
- moved R2 47.5 mm to (94.0, 20.0)
- moved C22 35.4 mm to (52.5, 54.0), turned to 90 degrees
- moved C21 35.4 mm to (2.50, 54.0), turned to 90 degrees
- moved C4 35.1 mm to (2.50, 4.48), turned to -90 degrees
- moved C6 35.1 mm to (102.5, 4.50), turned to 90 degrees
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Connections:
- C20 pad 1: Net-(J5-Pin_2) -> ANT1+
- C20 pad 2: GND -> ANT1+
- C21 pad 1: Net-(J6-Pin_2) -> ANT1+
- C21 pad 2: GND -> ANT1+
- C22 pad 1: Net-(J7-Pin_2) -> ANT1+
- C22 pad 2: GND -> ANT1+
- C23 pad 1: Net-(J8-Pin_2) -> ANT1+
- C23 pad 2: GND -> ANT1+
- C24 pad 1: Net-(J9-Pin_2) -> ANT1+
- C24 pad 2: GND -> ANT1+
- C25 pad 1: Net-(J10-Pin_2) -> ANT10+
- C25 pad 2: GND -> ANT10+
- C26 pad 1: Net-(J11-Pin_2) -> ANT10+
- C26 pad 2: GND -> ANT10+
- C27 pad 1: Net-(J12-Pin_2) -> ANT10+
- C27 pad 2: GND -> ANT10+
- C28 pad 1: Net-(J13-Pin_2) -> ANT10+
- C28 pad 2: GND -> ANT10+
- C29 pad 1: Net-(J14-Pin_2) -> ANT10+
- C29 pad 2: GND -> ANT10+
- C30 pad 1: Net-(J15-Pin_2) -> ANT10+
- C30 pad 2: GND -> ANT10+
- C31 pad 1: Net-(J16-Pin_2) -> ANT10+
- C31 pad 2: GND -> ANT10+
- C32 pad 1: Net-(J17-Pin_2) -> ANT10+
- C32 pad 2: GND -> ANT10+
- C33 pad 2: CLRC663.TX1 -> ANT1+
- C4 pad 1: Net-(J2-Pin_2) -> ANT1+
- C4 pad 2: GND -> ANT1+
- C5 pad 1: Net-(J3-Pin_2) -> ANT1+
- C5 pad 2: GND -> ANT1+
- C6 pad 1: Net-(J4-Pin_2) -> ANT1+
- C6 pad 2: GND -> ANT1+
- U1 pad 14: CLRC663.TX1 -> ANT1+
- U1 pad 18: CLRC663.RX -> ANT10+
- U5 pad 1: ANT8+ -> ANT1+
- U5 pad 13: ANT2+ -> ANT1+
- U5 pad 14: ANT3+ -> ANT1+
- U5 pad 15: ANT4+ -> ANT1+
- U5 pad 2: ANT7+ -> ANT1+
- U5 pad 3: CLRC663.TX1 -> ANT1+
- U5 pad 4: ANT6+ -> ANT1+
- U5 pad 5: ANT5+ -> ANT1+
- U7 pad 1: ANT16+ -> ANT10+
- U7 pad 12: ANT9+ -> ANT10+
- U7 pad 14: ANT11+ -> ANT10+
- U7 pad 15: ANT12+ -> ANT10+
- U7 pad 2: ANT15+ -> ANT10+
- U7 pad 3: CLRC663.RX -> ANT10+
- U7 pad 4: ANT14+ -> ANT10+
- U7 pad 5: ANT13+ -> ANT10+
Routing:
- net ANT1+: track 99.4 -> 7878.1 mm, vias 2 -> 46
- net ANT10+: track 46.0 -> 7523.7 mm, vias 2 -> 49
- net +5V: track 637.5 -> 76.6 mm, vias 8 -> 17
- net +3.3V: track 195.9 -> 40.3 mm, vias 5 -> 6
- net ANT16+: track 146.8 -> 0.00 mm
- net ANT4+: track 117.7 -> 0.00 mm, vias 2 -> 0
- net ANT13+: track 111.2 -> 0.00 mm, vias 2 -> 0
- net ANT8+: track 104.1 -> 0.00 mm
- net ANT9+: track 94.1 -> 0.00 mm, vias 2 -> 0
- net SCL: track 191.8 -> 98.0 mm
- net ANT3+: track 81.1 -> 0.00 mm, vias 2 -> 0
- net ANT14+: track 78.5 -> 0.00 mm, vias 2 -> 0
- net ANT2+: track 76.4 -> 0.00 mm, vias 2 -> 0
- net ANT15+: track 74.4 -> 0.00 mm, vias 2 -> 0
- net ANT5+: track 69.4 -> 0.00 mm, vias 2 -> 0
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Other:
- outline, holes or cut-outs redrawn
